Commit message: update urdf to fit ocs2 and urdf path

File: urdf/gen3_6dof_no_vision_urdf_arm.urdf (robot description, URDF)
Before this commit: robot gen3_6dof_no_vision_urdf_arm, 8 links, 7 joints
Links:
- link arm_base_link: geometry collision mesh filename=package://omni_mobile_manipulator/meshes/jaco/base_link.STL; visual mesh filename=package://omni_mobile_manipulator/meshes/jaco/base_link.STL
- link bicep_link: geometry collision mesh filename=package://omni_mobile_manipulator/meshes/jaco/bicep_link.STL; visual mesh filename=package://omni_mobile_manipulator/meshes/jaco/bicep_link.STL
- link bracelet_link: geometry collision mesh filename=package://omni_mobile_manipulator/meshes/jaco/bracelet_no_v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; visual mesh filename=package://omni_mobile_manipulator/meshes/jaco/bracelet_no_v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
- link forearm_link: geometry collision mesh filename=package://omni_mobile_manipulator/meshes/jaco/forearm_link.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; visual mesh filename=package://omni_mobile_manipulator/meshes/jaco/forearm_link.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
- link shoulder_link: geometry collision mesh filename=package://omni_mobile_manipulator/meshes/jaco/shoulder_link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; visual mesh filename=package://omni_mobile_manipulator/meshes/jaco/shoulder_link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
- link spherical_wrist_1_link: geometry collision mesh filename=package://omni_mobile_manipulator/meshes/jaco/spherical_wri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; visual mesh filename=package://omni_mobile_manipulator/meshes/jaco/spherical_wri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
- link spherical_wrist_2_link: geometry collision mesh filename=package://omni_mobile_manipulator/meshes/jaco/spherical_wri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; visual mesh filename=package://omni_mobile_manipulator/meshes/jaco/spherical_wri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

File: urdf/qxrobot_mm.urdf (robot description, URDF)
Before this commit: robot qxrobot_mm, 22 links, 21 joints
Links:
- added link base
- link arm_base_link: geometry collision mesh filename=package://omni_mobile_manipulator/meshes/jaco/base_link.STL; visual mesh filename=package://omni_mobile_manipulator/meshes/jaco/base_link.STL
- link base_link: geometry collision mesh filename=package://omni_mobile_manipulator/meshes/base_link.STL; visual mesh filename=package://omni_mobile_manipulator/meshes/base_link.STL
- link bicep_link: geometry collision mesh filename=package://omni_mobile_manipulator/meshes/jaco/bicep_link.STL; visual mesh filename=package://omni_mobile_manipulator/meshes/jaco/bicep_link.STL
- link bracelet_link: geometry collision mesh filename=package://omni_mobile_manipulator/meshes/jaco/bracelet_no_v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; visual mesh filename=package://omni_mobile_manipulator/meshes/jaco/bracelet_no_v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
- link camera_back_link: geometry collision mesh filename=package://omni_mobile_manipulator/meshes/camera_back_link.S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; visual mesh filename=package://omni_mobile_manipulator/meshes/camera_back_link.S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
- link camera_front_link: geometry collision mesh filename=package://omni_mobile_manipulator/meshes/camera_front_link.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; visual mesh filename=package://omni_mobile_manipulator/meshes/camera_front_link.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
- link forearm_link: geometry collision mesh filename=package://omni_mobile_manipulator/meshes/jaco/forearm_link.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; visual mesh filename=package://omni_mobile_manipulator/meshes/jaco/forearm_link.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
- link imu_link: geometry collision mesh filename=package://omni_mobile_manipulator/meshes/imu_link.STL; visual mesh filename=package://omni_mobile_manipulator/meshes/imu_link.STL
- link laser_link: geometry collision mesh filename=package://omni_mobile_manipulator/meshes/laser_link.STL; visual mesh filename=package://omni_mobile_manipulator/meshes/laser_link.STL
- link shoulder_link: geometry collision mesh filename=package://omni_mobile_manipulator/meshes/jaco/shoulder_link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; visual mesh filename=package://omni_mobile_manipulator/meshes/jaco/shoulder_link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
- link spherical_wrist_1_link: geometry collision mesh filename=package://omni_mobile_manipulator/meshes/jaco/spherical_wri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; visual mesh filename=package://omni_mobile_manipulator/meshes/jaco/spherical_wri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
- link spherical_wrist_2_link: geometry collision mesh filename=package://omni_mobile_manipulator/meshes/jaco/spherical_wri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; visual mesh filename=package://omni_mobile_manipulator/meshes/jaco/spherical_wri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
- link turn_back_left_link: geometry collision mesh filename=package://omni_mobile_manipulator/meshes/turn_back_left_lin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; visual mesh filename=package://omni_mobile_manipulator/meshes/turn_back_left_lin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
- link turn_back_right_link: geometry collision mesh filename=package://omni_mobile_manipulator/meshes/turn_back_right_li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; visual mesh filename=package://omni_mobile_manipulator/meshes/turn_back_right_li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
- link turn_front_left_link: geometry collision mesh filename=package://omni_mobile_manipulator/meshes/turn_front_left_li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; visual mesh filename=package://omni_mobile_manipulator/meshes/turn_front_left_li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
- link turn_front_right_link: geometry collision mesh filename=package://omni_mobile_manipulator/meshes/turn_front_right_l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; visual mesh filename=package://omni_mobile_manipulator/meshes/turn_front_right_l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
- link wheel_back_left_link: geometry collision mesh filename=package://omni_mobile_manipulator/meshes/wheel_back_left_li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; visual mesh filename=package://omni_mobile_manipulator/meshes/wheel_back_left_li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
- link wheel_back_right_link: geometry collision mesh filename=package://omni_mobile_manipulator/meshes/wheel_back_right_l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; visual mesh filename=package://omni_mobile_manipulator/meshes/wheel_back_right_l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
- link wheel_front_left_link: geometry collision mesh filename=package://omni_mobile_manipulator/meshes/wheel_front_left_l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; visual mesh filename=package://omni_mobile_manipulator/meshes/wheel_front_left_l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
- link wheel_front_right_link: geometry collision mesh filename=package://omni_mobile_manipulator/meshes/wheel_front_right_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; visual mesh filename=package://omni_mobile_manipulator/meshes/wheel_front_right_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
Joints:
- added joint world_to_base_link: type fixed, parent base, child base_link, origin xyz=0 0 0 rpy=0 0 0
- joint arm_joint: origin xyz=0.0 0 0.0 rpy=0 0 0 -> xyz=0.0 0.0 0.0 rpy=0 0 0
- joint joint_1: type continuous -> revolute
- joint joint_4: type continuous -> revolute
- joint joint_6: type continuous -> revolute
- joint turn_back_left_link_joint: axis 0 0 1 -> (none); limit lower=-9999 upper=9999 effort=9999 velocity=9999 -> (none); type continuous -> fixed
- joint turn_back_right_link_joint: axis 0 0 1 -> (none); limit lower=-9999 upper=9999 effort=9999 velocity=9999 -> (none); type continuous -> fixed
- joint turn_front_left_link_joint: limit lower=-9999 upper=9999 effort=9999 velocity=9999 -> lower=-3.14 upper=3.14 effort=150.0 velocity=1.3963; type continuous -> revolute
- joint turn_front_right_link_joint: axis 0 -1 0 -> (none); limit lower=-9999 upper=9999 effort=9999 velocity=9999 -> (none); type continuous -> fixed
- joint wheel_back_left_link_joint: axis 0 -1 0 -> (none); limit lower=-9999 upper=9999 effort=9999 velocity=9999 -> (none); type continuous -> fixed
- joint wheel_back_right_link_joint: axis 0 1 0 -> (none); limit lower=-9999 upper=9999 effort=9999 velocity=9999 -> (none); type continuous -> fixed
- joint wheel_front_left_link_joint: axis 0 1 0 -> (none); limit lower=-9999 upper=9999 effort=9999 velocity=9999 -> (none); type continuous -> fixed
- joint wheel_front_right_link_joint: axis 0 -1 0 -> (none); limit lower=-9999 upper=9999 effort=9999 velocity=9999 -> (none); type continuous -> fixed

File: urdf/qxrobot_urdf_v1.urdf (robot description, URDF)
Before this commit: robot qxrobot_urdf_v1, 14 links, 13 joints
Links:
- link base_link: geometry collision mesh filename=package://omni_mobile_manipulator/meshes/base_link.STL; visual mesh filename=package://omni_mobile_manipulator/meshes/base_link.STL
- link camera_back_link: geometry collision mesh filename=package://omni_mobile_manipulator/meshes/camera_back_link.S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; visual mesh filename=package://omni_mobile_manipulator/meshes/camera_back_link.S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
- link camera_front_link: geometry collision mesh filename=package://omni_mobile_manipulator/meshes/camera_front_link.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; visual mesh filename=package://omni_mobile_manipulator/meshes/camera_front_link.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
- link imu_link: geometry collision mesh filename=package://omni_mobile_manipulator/meshes/imu_link.STL; visual mesh filename=package://omni_mobile_manipulator/meshes/imu_link.STL
- link laser_link: geometry collision mesh filename=package://omni_mobile_manipulator/meshes/laser_link.STL; visual mesh filename=package://omni_mobile_manipulator/meshes/laser_link.STL
- link turn_back_left_link: geometry collision mesh filename=package://omni_mobile_manipulator/meshes/turn_back_left_lin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; visual mesh filename=package://omni_mobile_manipulator/meshes/turn_back_left_lin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
- link turn_back_right_link: geometry collision mesh filename=package://omni_mobile_manipulator/meshes/turn_back_right_li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; visual mesh filename=package://omni_mobile_manipulator/meshes/turn_back_right_li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
- link turn_front_left_link: geometry collision mesh filename=package://omni_mobile_manipulator/meshes/turn_front_left_li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; visual mesh filename=package://omni_mobile_manipulator/meshes/turn_front_left_li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
- link turn_front_right_link: geometry collision mesh filename=package://omni_mobile_manipulator/meshes/turn_front_right_l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; visual mesh filename=package://omni_mobile_manipulator/meshes/turn_front_right_l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
- link wheel_back_left_link: geometry collision mesh filename=package://omni_mobile_manipulator/meshes/wheel_back_left_li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; visual mesh filename=package://omni_mobile_manipulator/meshes/wheel_back_left_li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
- link wheel_back_right_link: geometry collision mesh filename=package://omni_mobile_manipulator/meshes/wheel_back_right_l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; visual mesh filename=package://omni_mobile_manipulator/meshes/wheel_back_right_l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
- link wheel_front_left_link: geometry collision mesh filename=package://omni_mobile_manipulator/meshes/wheel_front_left_l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; visual mesh filename=package://omni_mobile_manipulator/meshes/wheel_front_left_l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
- link wheel_front_right_link: geometry collision mesh filename=package://omni_mobile_manipulator/meshes/wheel_front_right_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; visual mesh filename=package://omni_mobile_manipulator/meshes/wheel_front_right_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

File: urdf/xacro/gen3_macro.xacro (robot description, xacro)
@@ -13,14 +13,14 @@
         <origin xyz="0 0 0" rpy="0 0 0" />
         <geometry>
-          <mesh filename="package://qxrobot_urdf_v1/meshes/jaco/base_link.STL" />
-        </geometry>
-        <material name="">
-          <color rgba="0.75294 0.75294 0.75294 1" />
-        </material>
-      </visual>
-      <collision>
-        <origin xyz="0 0 0" rpy="0 0 0" />
-        <geometry>
-          <mesh filename="package://qxrobot_urdf_v1/meshes/jaco/base_link.STL" />
+          <mesh filename="package://omni_mobile_manipulator/meshes/jaco/base_link.STL" />
+        </geometry>
+        <material name="">
+          <color rgba="0.75294 0.75294 0.75294 1" />
+        </material>
+      </visual>
+      <collision>
+        <origin xyz="0 0 0" rpy="0 0 0" />
+        <geometry>
+          <mesh filename="package://omni_mobile_manipulator/meshes/jaco/base_link.STL" />
         </geometry>
       </collision>
@@ -35,14 +35,14 @@
         <origin xyz="0 0 0" rpy="0 0 0" />
         <geometry>
-          <mesh filename="package://qxrobot_urdf_v1/meshes/jaco/shoulder_link.STL" />
-        </geometry>
-        <material name="">
-          <color rgba="0.75294 0.75294 0.75294 1" />
-        </material>
-      </visual>
-      <collision>
-        <origin xyz="0 0 0" rpy="0 0 0" />
-        <geometry>
-          <mesh filename="package://qxrobot_urdf_v1/meshes/jaco/shoulder_link.STL" />
+          <mesh filename="package://omni_mobile_manipulator/meshes/jaco/shoulder_link.STL" />
+        </geometry>
+        <material name="">
+          <color rgba="0.75294 0.75294 0.75294 1" />
+        </material>
+      </visual>
+      <collision>
+        <origin xyz="0 0 0" rpy="0 0 0" />
+        <geometry>
+          <mesh filename="package://omni_mobile_manipulator/meshes/jaco/shoulder_link.STL" />
         </geometry>
       </collision>
@@ -64,14 +64,14 @@
         <origin xyz="0 0 0" rpy="0 0 0" />
         <geometry>
-          <mesh filename="package://qxrobot_urdf_v1/meshes/jaco/bicep_link.STL" />
-        </geometry>
-        <material name="">
-          <color rgba="0.75294 0.75294 0.75294 1" />
-        </material>
-      </visual>
-      <collision>
-        <origin xyz="0 0 0" rpy="0 0 0" />
-        <geometry>
-          <mesh filename="package://qxrobot_urdf_v1/meshes/jaco/bicep_link.STL" />
+          <mesh filename="package://omni_mobile_manipulator/meshes/jaco/bicep_link.STL" />
+        </geometry>
+        <material name="">
+          <color rgba="0.75294 0.75294 0.75294 1" />
+        </material>
+      </visual>
+      <collision>
+        <origin xyz="0 0 0" rpy="0 0 0" />
+        <geometry>
+          <mesh filename="package://omni_mobile_manipulator/meshes/jaco/bicep_link.STL" />
         </geometry>
       </collision>
@@ -93,14 +93,14 @@
         <origin xyz="0 0 0" rpy="0 0 0" />
         <geometry>
-          <mesh filename="package://qxrobot_urdf_v1/meshes/jaco/forearm_link.STL" />
-        </geometry>
-        <material name="">
-          <color rgba="0.75294 0.75294 0.75294 1" />
-        </material>
-      </visual>
-      <collision>
-        <origin xyz="0 0 0" rpy="0 0 0" />
-        <geometry>
-          <mesh filename="package://qxrobot_urdf_v1/meshes/jaco/forearm_link.STL" />
+          <mesh filename="package://omni_mobile_manipulator/meshes/jaco/forearm_link.STL" />
+        </geometry>
+        <material name="">
+          <color rgba="0.75294 0.75294 0.75294 1" />
+        </material>
+      </visual>
+      <collision>
+        <origin xyz="0 0 0" rpy="0 0 0" />
+        <geometry>
+          <mesh filename="package://omni_mobile_manipulator/meshes/jaco/forearm_link.STL" />
         </geometry>
       </collision>
@@ -122,14 +122,14 @@
         <origin xyz="0 0 0" rpy="0 0 0" />
         <geometry>
-          <mesh filename="package://qxrobot_urdf_v1/meshes/jaco/spherical_wrist_1_link.STL" />
-        </geometry>
-        <material name="">
-          <color rgba="0.75294 0.75294 0.75294 1" />
-        </material>
-      </visual>
-      <collision>
-        <origin xyz="0 0 0" rpy="0 0 0" />
-        <geometry>
-          <mesh filename="package://qxrobot_urdf_v1/meshes/jaco/spherical_wrist_1_link.STL" />
+          <mesh filename="package://omni_mobile_manipulator/meshes/jaco/spherical_wrist_1_link.STL" />
+        </geometry>
+        <material name="">
+          <color rgba="0.75294 0.75294 0.75294 1" />
+        </material>
+      </visual>
+      <collision>
+        <origin xyz="0 0 0" rpy="0 0 0" />
+        <geometry>
+          <mesh filename="package://omni_mobile_manipulator/meshes/jaco/spherical_wrist_1_link.STL" />
         </geometry>
       </collision>
@@ -151,14 +151,14 @@
         <origin xyz="0 0 0" rpy="0 0 0" />
         <geometry>
-          <mesh filename="package://qxrobot_urdf_v1/meshes/jaco/spherical_wrist_2_link.STL" />
-        </geometry>
-        <material name="">
-          <color rgba="0.75294 0.75294 0.75294 1" />
-        </material>
-      </visual>
-      <collision>
-        <origin xyz="0 0 0" rpy="0 0 0" />
-        <geometry>
-          <mesh filename="package://qxrobot_urdf_v1/meshes/jaco/spherical_wrist_2_link.STL" />
+          <mesh filename="package://omni_mobile_manipulator/meshes/jaco/spherical_wrist_2_link.STL" />
+        </geometry>
+        <material name="">
+          <color rgba="0.75294 0.75294 0.75294 1" />
+        </material>
+      </visual>
+      <collision>
+        <origin xyz="0 0 0" rpy="0 0 0" />
+        <geometry>
+          <mesh filename="package://omni_mobile_manipulator/meshes/jaco/spherical_wrist_2_link.STL" />
         </geometry>
       </collision>
@@ -181,14 +181,14 @@
         <origin xyz="0 0 0" rpy="0 0 0" />
         <geometry>
-          <mesh filename="package://qxrobot_urdf_v1/meshes/jaco/bracelet_with_vision_link.STL" />
-        </geometry>
-        <material name="">
-          <color rgba="0.75294 0.75294 0.75294 1" />
-        </material>
-      </visual>
-      <collision>
-        <origin xyz="0 0 0" rpy="0 0 0" />
-        <geometry>
-          <mesh filename="package://qxrobot_urdf_v1/meshes/jaco/bracelet_with_vision_link.STL" />
+          <mesh filename="package://omni_mobile_manipulator/meshes/jaco/bracelet_with_vision_link.STL" />
+        </geometry>
+        <material name="">
+          <color rgba="0.75294 0.75294 0.75294 1" />
+        </material>
+      </visual>
+      <collision>
+        <origin xyz="0 0 0" rpy="0 0 0" />
+        <geometry>
+          <mesh filename="package://omni_mobile_manipulator/meshes/jaco/bracelet_with_vision_link.STL" />
         </geometry>
       </collision>
@@ -205,14 +205,14 @@
         <origin xyz="0 0 0" rpy="0 0 0" />
         <geometry>
-          <mesh filename="package://qxrobot_urdf_v1/meshes/jaco/bracelet_no_vision_link.STL" />
-        </geometry>
-        <material name="">
-          <color rgba="0.75294 0.75294 0.75294 1" />
-        </material>
-      </visual>
-      <collision>
-        <origin xyz="0 0 0" rpy="0 0 0" />
-        <geometry>
-          <mesh filename="package://qxrobot_urdf_v1/meshes/jaco/bracelet_no_vision_link.STL" />
+          <mesh filename="package://omni_mobile_manipulator/meshes/jaco/bracelet_no_vision_link.STL" />
+        </geometry>
+        <material name="">
+          <color rgba="0.75294 0.75294 0.75294 1" />
+        </material>
+      </visual>
+      <collision>
+        <origin xyz="0 0 0" rpy="0 0 0" />
+        <geometry>
+          <mesh filename="package://omni_mobile_manipulator/meshes/jaco/bracelet_no_vision_link.STL" />
         </geometry>
       </collision>

File: urdf/xacro/qxrobot_mm.xacro (robot description, xacro)
@@ -9,14 +9,14 @@
     <xacro:macro name="load_robot" params="gripper dof vision sim prefix gazebo">
         <!-- Files to include -->
-        <xacro:include filename="$(find qxrobot_urdf_v1)/urdf/xacro/gen3_macro.xacro" />
+        <xacro:include filename="$(find omni_mobile_manipulator)/urdf/xacro/gen3_macro.xacro" />
         <xacro:unless value="${not gripper}">
-            <xacro:include filename="$(find qxrobot_urdf_v1)/urdf/xacro/${gripper}_macro.xacro" />
+            <xacro:include filename="$(find omni_mobile_manipulator)/urdf/xacro/${gripper}_macro.xacro" />
         </xacro:unless>
         <xacro:if value="${sim}">
             <!-- Arm transmission elements-->
-            <xacro:include filename="$(find qxrobot_urdf_v1)/urdf/xacro/gen3_transmission_macro.xacro" />
+            <xacro:include filename="$(find omni_mobile_manipulator)/urdf/xacro/gen3_transmission_macro.xacro" />
             <!-- Gripper transmission elements if there is a gripper-->
             <xacro:unless value="${not gripper}">
-                <xacro:include filename="$(find qxrobot_urdf_v1)/urdf/xacro/${gripper}_transmission_macro.xacro" />
+                <xacro:include filename="$(find omni_mobile_manipulator)/urdf/xacro/${gripper}_transmission_macro.xacro" />
             </xacro:unless>
         </xacro:if>
@@ -63,5 +63,5 @@
     </xacro:macro>
     <xacro:load_robot gripper="$(arg gripper)" dof="$(arg dof)" vision="$(arg vision)" sim="$(arg sim)" prefix="$(arg prefix)" gazebo="$(arg gazebo)" />
-    <xacro:include filename="$(find qxrobot_urdf_v1)/urdf/xacro/qxrobot_urdf_v1.xacro" />
+    <xacro:include filename="$(find omni_mobile_manipulator)/urdf/xacro/omni_mobile_manipulator.xacro" />
     <xacro:load_base/>
     <joint name="base_footprint_joint" type="fixed">
