Commit message: update urdf to fit ocs2 and urdf path

File: urdf/xacro/qxrobot_urdf_v1.xacro (robot description, xacro)
@@ -3,5 +3,5 @@
      Commit Version: 1.5.1-0-g916b5db  Build Version: 1.5.7152.31018
      For more information, please see http://wiki.ros.org/sw_urdf_exporter -->
-<robot name="qxrobot_urdf_v1" xmlns:xacro="http://ros.org/wiki/xacro">
+<robot name="omni_mobile_manipulator" xmlns:xacro="http://ros.org/wiki/xacro">
 <xacro:macro name="load_base" params="">
   <link
@@ -27,5 +27,5 @@
       <geometry>
         <mesh
-          filename="package://qxrobot_urdf_v1/meshes/base_link.STL" />
+          filename="package://omni_mobile_manipulator/meshes/base_link.STL" />
       </geometry>
       <material
@@ -41,5 +41,5 @@
       <geometry>
         <mesh
-          filename="package://qxrobot_urdf_v1/meshes/base_link.STL" />
+          filename="package://omni_mobile_manipulator/meshes/base_link.STL" />
       </geometry>
     </collision>
@@ -67,5 +67,5 @@
       <geometry>
         <mesh
-          filename="package://qxrobot_urdf_v1/meshes/turn_front_left_link.STL" />
+          filename="package://omni_mobile_manipulator/meshes/turn_front_left_link.STL" />
       </geometry>
       <material
@@ -81,5 +81,5 @@
       <geometry>
         <mesh
-          filename="package://qxrobot_urdf_v1/meshes/turn_front_left_link.STL" />
+          filename="package://omni_mobile_manipulator/meshes/turn_front_left_link.STL" />
       </geometry>
     </collision>
@@ -127,5 +127,5 @@
       <geometry>
         <mesh
-          filename="package://qxrobot_urdf_v1/meshes/wheel_front_left_link.STL" />
+          filename="package://omni_mobile_manipulator/meshes/wheel_front_left_link.STL" />
       </geometry>
       <material
@@ -141,5 +141,5 @@
       <geometry>
         <mesh
-          filename="package://qxrobot_urdf_v1/meshes/wheel_front_left_link.STL" />
+          filename="package://omni_mobile_manipulator/meshes/wheel_front_left_link.STL" />
       </geometry>
     </collision>
@@ -187,5 +187,5 @@
       <geometry>
         <mesh
-          filename="package://qxrobot_urdf_v1/meshes/turn_front_right_link.STL" />
+          filename="package://omni_mobile_manipulator/meshes/turn_front_right_link.STL" />
       </geometry>
       <material
@@ -201,5 +201,5 @@
       <geometry>
         <mesh
-          filename="package://qxrobot_urdf_v1/meshes/turn_front_right_link.STL" />
+          filename="package://omni_mobile_manipulator/meshes/turn_front_right_link.STL" />
       </geometry>
     </collision>
@@ -247,5 +247,5 @@
       <geometry>
         <mesh
-          filename="package://qxrobot_urdf_v1/meshes/wheel_front_right_link.STL" />
+          filename="package://omni_mobile_manipulator/meshes/wheel_front_right_link.STL" />
       </geometry>
       <material
@@ -261,5 +261,5 @@
       <geometry>
         <mesh
-          filename="package://qxrobot_urdf_v1/meshes/wheel_front_right_link.STL" />
+          filename="package://omni_mobile_manipulator/meshes/wheel_front_right_link.STL" />
       </geometry>
     </collision>
@@ -307,5 +307,5 @@
       <geometry>
         <mesh
-          filename="package://qxrobot_urdf_v1/meshes/turn_back_left_link.STL" />
+          filename="package://omni_mobile_manipulator/meshes/turn_back_left_link.STL" />
       </geometry>
       <material
@@ -321,5 +321,5 @@
       <geometry>
         <mesh
-          filename="package://qxrobot_urdf_v1/meshes/turn_back_left_link.STL" />
+          filename="package://omni_mobile_manipulator/meshes/turn_back_left_link.STL" />
       </geometry>
     </collision>
@@ -367,5 +367,5 @@
       <geometry>
         <mesh
-          filename="package://qxrobot_urdf_v1/meshes/wheel_back_left_link.STL" />
+          filename="package://omni_mobile_manipulator/meshes/wheel_back_left_link.STL" />
       </geometry>
       <material
@@ -381,5 +381,5 @@
       <geometry>
         <mesh
-          filename="package://qxrobot_urdf_v1/meshes/wheel_back_left_link.STL" />
+          filename="package://omni_mobile_manipulator/meshes/wheel_back_left_link.STL" />
       </geometry>
     </collision>
@@ -427,5 +427,5 @@
       <geometry>
         <mesh
-          filename="package://qxrobot_urdf_v1/meshes/turn_back_right_link.STL" />
+          filename="package://omni_mobile_manipulator/meshes/turn_back_right_link.STL" />
       </geometry>
       <material
@@ -441,5 +441,5 @@
       <geometry>
         <mesh
-          filename="package://qxrobot_urdf_v1/meshes/turn_back_right_link.STL" />
+          filename="package://omni_mobile_manipulator/meshes/turn_back_right_link.STL" />
       </geometry>
     </collision>
@@ -487,5 +487,5 @@
       <geometry>
         <mesh
-          filename="package://qxrobot_urdf_v1/meshes/wheel_back_right_link.STL" />
+          filename="package://omni_mobile_manipulator/meshes/wheel_back_right_link.STL" />
       </geometry>
       <material
@@ -501,5 +501,5 @@
       <geometry>
         <mesh
-          filename="package://qxrobot_urdf_v1/meshes/wheel_back_right_link.STL" />
+          filename="package://omni_mobile_manipulator/meshes/wheel_back_right_link.STL" />
       </geometry>
     </collision>
@@ -545,5 +545,5 @@
       <geometry>
         <mesh
-          filename="package://qxrobot_urdf_v1/meshes/camera_front_link.STL" />
+          filename="package://omni_mobile_manipulator/meshes/camera_front_link.STL" />
       </geometry>
       <material
@@ -559,5 +559,5 @@
       <geometry>
         <mesh
-          filename="package://qxrobot_urdf_v1/meshes/camera_front_link.STL" />
+          filename="package://omni_mobile_manipulator/meshes/camera_front_link.STL" />
       </geometry>
     </collision>
@@ -598,5 +598,5 @@
       <geometry>
         <mesh
-          filename="package://qxrobot_urdf_v1/meshes/camera_back_link.STL" />
+          filename="package://omni_mobile_manipulator/meshes/camera_back_link.STL" />
       </geometry>
       <material
@@ -612,5 +612,5 @@
       <geometry>
         <mesh
-          filename="package://qxrobot_urdf_v1/meshes/camera_back_link.STL" />
+          filename="package://omni_mobile_manipulator/meshes/camera_back_link.STL" />
       </geometry>
     </collision>
@@ -651,5 +651,5 @@
       <geometry>
         <mesh
-          filename="package://qxrobot_urdf_v1/meshes/imu_link.STL" />
+          filename="package://omni_mobile_manipulator/meshes/imu_link.STL" />
       </geometry>
       <material
@@ -665,5 +665,5 @@
       <geometry>
         <mesh
-          filename="package://qxrobot_urdf_v1/meshes/imu_link.STL" />
+          filename="package://omni_mobile_manipulator/meshes/imu_link.STL" />
       </geometry>
     </collision>
@@ -704,5 +704,5 @@
       <geometry>
         <mesh
-          filename="package://qxrobot_urdf_v1/meshes/laser_link.STL" />
+          filename="package://omni_mobile_manipulator/meshes/laser_link.STL" />
       </geometry>
       <material
@@ -718,5 +718,5 @@
       <geometry>
         <mesh
-          filename="package://qxrobot_urdf_v1/meshes/laser_link.STL" />
+          filename="package://omni_mobile_manipulator/meshes/laser_link.STL" />
       </geometry>
     </collision>

File: urdf/xacro/robotiq_2f_85_macro.xacro (robot description, xacro)
@@ -2,5 +2,5 @@
 <robot name="robotiq_arg2f_85_model" xmlns:xacro="http://ros.org/wiki/xacro">
   <xacro:macro name="load_gripper" params="parent prefix">
-    <xacro:include filename="$(find qxrobot_urdf_v1)/urdf/xacro/robotiq_arg2f_85_model_macro.xacro" />
+    <xacro:include filename="$(find omni_mobile_manipulator)/urdf/xacro/robotiq_arg2f_85_model_macro.xacro" />
     <xacro:robotiq_arg2f_85 parent="${parent}" prefix="${prefix}"/>
   </xacro:macro>

File: urdf/xacro/robotiq_arg2f.xacro (robot description, xacro)
@@ -19,5 +19,5 @@
           <!-- The DAE file doesn't show well in Gazebo so we're using the STL instead -->
           <!-- <mesh filename="package://kortex_description/grippers/robotiq_2f_85/meshes/visual/robotiq_arg2f_85_base_link.dae" scale="0.001 0.001 0.001"/> -->
-          <mesh filename="package://qxrobot_urdf_v1/meshes/gripper/collision/robotiq_arg2f_base_link.stl" />
+          <mesh filename="package://omni_mobile_manipulator/meshes/gripper/collision/robotiq_arg2f_base_link.stl" />
         </geometry>
         <material name="">
@@ -28,5 +28,5 @@
         <origin xyz="0 0 0" rpy="0 0 0" />
         <geometry>
-           <mesh filename="package://qxrobot_urdf_v1/meshes/gripper/collision/robotiq_arg2f_base_link.stl" />
+           <mesh filename="package://omni_mobile_manipulator/meshes/gripper/collision/robotiq_arg2f_base_link.stl" />
         </geometry>
       </collision>

File: urdf/xacro/robotiq_arg2f_85_model_macro.xacro (robot description, xacro)
@@ -13,5 +13,5 @@
         <origin xyz="0 0 0" rpy="0 0 0" />
         <geometry>
-          <mesh filename="package://qxrobot_urdf_v1/meshes/gripper/visual/robotiq_arg2f_85_outer_knuckle.dae" scale="0.001 0.001 0.001"/>
+          <mesh filename="package://omni_mobile_manipulator/meshes/gripper/visual/robotiq_arg2f_85_outer_knuckle.dae" scale="0.001 0.001 0.001"/>
         </geometry>
         <material name="">
@@ -22,5 +22,5 @@
         <origin xyz="0 0 0" rpy="0 0 0" />
         <geometry>
-          <mesh filename="package://qxrobot_urdf_v1/meshes/gripper/collision/robotiq_arg2f_85_outer_knuckle.dae" scale="0.001 0.001 0.001"/>
+          <mesh filename="package://omni_mobile_manipulator/meshes/gripper/collision/robotiq_arg2f_85_outer_knuckle.dae" scale="0.001 0.001 0.001"/>
         </geometry>
       </collision>
@@ -37,5 +37,5 @@
         <origin xyz="0 0 0" rpy="0 0 0" />
         <geometry>
-          <mesh filename="package://qxrobot_urdf_v1/meshes/gripper/visual/robotiq_arg2f_85_outer_finger.dae" scale="0.001 0.001 0.001"/>
+          <mesh filename="package://omni_mobile_manipulator/meshes/gripper/visual/robotiq_arg2f_85_outer_finger.dae" scale="0.001 0.001 0.001"/>
         </geometry>
         <material name="">
@@ -46,5 +46,5 @@
         <origin xyz="0 0 0" rpy="0 0 0" />
         <geometry>
-          <mesh filename="package://qxrobot_urdf_v1/meshes/gripper/collision/robotiq_arg2f_85_outer_finger.dae" scale="0.001 0.001 0.001"/>
+          <mesh filename="package://omni_mobile_manipulator/meshes/gripper/collision/robotiq_arg2f_85_outer_finger.dae" scale="0.001 0.001 0.001"/>
         </geometry>
       </collision>
@@ -61,5 +61,5 @@
         <origin xyz="0 0 0" rpy="0 0 0" />
         <geometry>
-          <mesh filename="package://qxrobot_urdf_v1/meshes/gripper/visual/robotiq_arg2f_85_inner_knuckle.dae" scale="0.001 0.001 0.001"/>
+          <mesh filename="package://omni_mobile_manipulator/meshes/gripper/visual/robotiq_arg2f_85_inner_knuckle.dae" scale="0.001 0.001 0.001"/>
         </geometry>
         <material name="">
@@ -70,5 +70,5 @@
         <origin xyz="0 0 0" rpy="0 0 0" />
         <geometry>
-          <mesh filename="package://qxrobot_urdf_v1/meshes/gripper/collision/robotiq_arg2f_85_inner_knuckle.dae" scale="0.001 0.001 0.001"/>
+          <mesh filename="package://omni_mobile_manipulator/meshes/gripper/collision/robotiq_arg2f_85_inner_knuckle.dae" scale="0.001 0.001 0.001"/>
         </geometry>
       </collision>
@@ -85,5 +85,5 @@
         <origin xyz="0 0 0" rpy="0 0 0" />
         <geometry>
-          <mesh filename="package://qxrobot_urdf_v1/meshes/gripper/visual/robotiq_arg2f_85_inner_finger.dae" scale="0.001 0.001 0.001"/>
+          <mesh filename="package://omni_mobile_manipulator/meshes/gripper/visual/robotiq_arg2f_85_inner_finger.dae" scale="0.001 0.001 0.001"/>
         </geometry>
         <material name="">
@@ -94,5 +94,5 @@
         <origin xyz="0 0 0" rpy="0 0 0" />
         <geometry>
-          <mesh filename="package://qxrobot_urdf_v1/meshes/gripper/collision/robotiq_arg2f_85_inner_finger.dae" scale="0.001 0.001 0.001" />
+          <mesh filename="package://omni_mobile_manipulator/meshes/gripper/collision/robotiq_arg2f_85_inner_finger.dae" scale="0.001 0.001 0.001" />
         </geometry>
       </collision>
@@ -159,5 +159,5 @@
     </joint>
   </xacro:macro>
-  <xacro:include filename="$(find qxrobot_urdf_v1)/urdf/xacro/robotiq_arg2f.xacro" />
+  <xacro:include filename="$(find omni_mobile_manipulator)/urdf/xacro/robotiq_arg2f.xacro" />
   <xacro:macro name="finger_joint" params="prefix">
     <joint name="${prefix}finger_joint" type="revolute">
